File: doorbell-adapter.sch (KiCad schematic (older format))
At the start: 12 parts, among them U1 TLP185

Commit message: Finish PCB
Parts:
- removed U1: TLP185, Package_SO:SOIC-4_4.55x3.7mm_P2.54mm, symbol Isolator:TLP185
- added H1: MountingHole, extraFootprints:MountingHole_3.2mm_M3_ISO7380_Keepout, symbol Mechanical:MountingHole
- added U1: PC817, Package_DIP:DIP-4_W7.62mm, symbol Isolator:PC817
- D1, D2, D3, D4: footprint Diode_SMD:D_0603_1608Metric -> Diode_SMD:D_SOD-523
- R1: value R -> 18k
- R2: value R -> 100R
- R3: value R -> 2k
Connections:
- net GND: now also U1.2
- net at J_ESP1.1 (Pin_1): now also U1.4
- net at J_ESP1.2 (Pin_2): now also U1.3
- net at R2.2: now also U1.1
Changed lines of the file:
@@
 U 1 1 619F5EAD
 P 6150 3200
-F 0 "J_Bell1" H 6150 3300 50  0000 R CNN
-F 1 "Molex PicoBlade 2Pin" H 6122 3083 50  0000 R CNN
+F 0 "J_Bell1" V 6200 3500 50  0000 R CNN
+F 1 "Molex PicoBlade 2Pin" V 6050 3500 50  0000 R CNN
 F 2 "Connector_Molex:Molex_PicoBlade_53047-0210_1x02_P1.25mm_Vertical" H 6150 3200 50  0001 C CNN
 F 3 "~" H 6150 3200 50  0001 C CNN
@@
 U 1 1 619F69A3
 P 2250 3300
-F 0 "J_ESP1" H 2358 3481 50  0000 C CNN
-F 1 "Molex PicoBlade 2Pin" H 2358 3390 50  0000 C CNN
+F 0 "J_ESP1" H 2400 3500 50  0000 C CNN
+F 1 "Molex PicoBlade 2Pin" V 2150 3300 50  0000 C CNN
 F 2 "Connector_Molex:Molex_PicoBlade_53047-0210_1x02_P1.25mm_Vertical" H 2250 3300 50  0001 C CNN
 F 3 "~" H 2250 3300 50  0001 C CNN
@@
 F 0 "D1" H 5400 3017 50  0000 C CNN
 F 1 "D" H 5400 2926 50  0000 C CNN
-F 2 "Diode_SMD:D_0603_1608Metric" H 5400 2800 50  0001 C CNN
+F 2 "Diode_SMD:D_SOD-523" H 5400 2800 50  0001 C CNN
 F 3 "~" H 5400 2800 50  0001 C CNN
 	1    5400 2800
@@
 F 0 "D2" V 5104 3130 50  0000 L CNN
 F 1 "D" V 5195 3130 50  0000 L CNN
-F 2 "Diode_SMD:D_0603_1608Metric" H 5150 3050 50  0001 C CNN
+F 2 "Diode_SMD:D_SOD-523" H 5150 3050 50  0001 C CNN
 F 3 "~" H 5150 3050 50  0001 C CNN
 	1    5150 3050
@@
 F 0 "D4" H 5400 3083 50  0000 C CNN
 F 1 "D" H 5400 3174 50  0000 C CNN
-F 2 "Diode_SMD:D_0603_1608Metric" H 5400 3300 50  0001 C CNN
+F 2 "Diode_SMD:D_SOD-523" H 5400 3300 50  0001 C CNN
 F 3 "~" H 5400 3300 50  0001 C CNN
 	1    5400 3300
@@
 F 0 "D3" V 5604 2970 50  0000 R CNN
 F 1 "D" V 5695 2970 50  0000 R CNN
-F 2 "Diode_SMD:D_0603_1608Metric" H 5650 3050 50  0001 C CNN
+F 2 "Diode_SMD:D_SOD-523" H 5650 3050 50  0001 C CNN
 F 3 "~" H 5650 3050 50  0001 C CNN
 	1    5650 3050
@@
 P 4400 3400
 F 0 "R3" H 4470 3446 50  0000 L CNN
-F 1 "R" H 4470 3355 50  0000 L CNN
+F 1 "2k" H 4470 3355 50  0000 L CNN
 F 2 "Resistor_SMD:R_0603_1608Metric" V 4330 3400 50  0001 C CNN
 F 3 "~" H 4400 3400 50  0001 C CNN
@@
 P 4400 3000
 F 0 "R1" H 4470 3046 50  0000 L CNN
-F 1 "R" H 4470 2955 50  0000 L CNN
+F 1 "18k" H 4470 2955 50  0000 L CNN
 F 2 "Resistor_SMD:R_0603_1608Metric" V 4330 3000 50  0001 C CNN
 F 3 "~" H 4400 3000 50  0001 C CNN
@@
 Wire Wire Line
 	4400 3200 4400 3250
-$Comp
-L Isolator:TLP185 U1
-U 1 1 61A025A2
-P 3200 3300
-F 0 "U1" H 3200 3625 50  0000 C CNN
-F 1 "TLP185" H 3200 3534 50  0000 C CNN
-F 2 "Package_SO:SOIC-4_4.55x3.7mm_P2.54mm" H 3200 3000 50  0001 C CIN
-F 3 "https://toshiba.semicon-storage.com/info/docget.jsp?did=11791&prodName=TLP185" H 3200 3300 50  0001 L CNN
-	1    3200 3300
-	-1   0    0    -1
-$EndComp
 $Comp
 L Device:C C1
@@
 P 3800 3200
 F 0 "R2" V 3593 3200 50  0000 C CNN
-F 1 "R" V 3684 3200 50  0000 C CNN
+F 1 "100R" V 3684 3200 50  0000 C CNN
 F 2 "Resistor_SMD:R_0603_1608Metric" V 3730 3200 50  0001 C CNN
 F 3 "~" H 3800 3200 50  0001 C CNN
@@
 Wire Wire Line
 	2450 3400 2900 3400
+$Comp
+L power:PWR_FLAG #FLG0101
+U 1 1 61A1524C
+P 4750 2600
+F 0 "#FLG0101" H 4750 2675 50  0001 C CNN
+F 1 "PWR_FLAG" H 4750 2773 50  0000 C CNN
+F 2 "" H 4750 2600 50  0001 C CNN
+F 3 "~" H 4750 2600 50  0001 C CNN
+	1    4750 2600
+	1    0    0    -1
+$EndComp
+Wire Wire Line
+	4750 2600 4750 2800
+$Comp
+L power:PWR_FLAG #FLG0102
+U 1 1 61A1629A
+P 4750 3750
+F 0 "#FLG0102" H 4750 3825 50  0001 C CNN
+F 1 "PWR_FLAG" H 4750 3923 50  0000 C CNN
+F 2 "" H 4750 3750 50  0001 C CNN
+F 3 "~" H 4750 3750 50  0001 C CNN
+	1    4750 3750
+	-1   0    0    1
+$EndComp
+Wire Wire Line
+	4750 3600 4750 3750
+$Comp
+L Isolator:PC817 U1
+U 1 1 61A1A9E6
+P 3200 3300
+F 0 "U1" H 3200 3625 50  0000 C CNN
+F 1 "PC817" H 3200 3534 50  0000 C CNN
+F 2 "Package_DIP:DIP-4_W7.62mm" H 3000 3100 50  0001 L CIN
+F 3 "http://www.soselectronic.cz/a_info/resource/d/pc817.pdf" H 3200 3300 50  0001 L CNN
+	1    3200 3300
+	-1   0    0    -1
+$EndComp
+Wire Notes Line
+	2050 2350 6350 2350
+Wire Notes Line
+	6350 2350 6350 4000
+Wire Notes Line
+	6350 4000 2050 4000
+Wire Notes Line
+	2050 2350 2050 4000
+$Comp
+L Mechanical:MountingHole H1
+U 1 1 61A1F7EE
+P 2200 2050
+F 0 "H1" H 2300 2096 50  0000 L CNN
+F 1 "MountingHole" H 2300 2005 50  0000 L CNN
+F 2 "extraFootprints:MountingHole_3.2mm_M3_ISO7380_Keepout" H 2200 2050 50  0001 C CNN
+F 3 "~" H 2200 2050 50  0001 C CNN
+	1    2200 2050
+	1    0    0    -1
+$EndComp
+Wire Notes Line
+	2050 1900 2050 2250
+Wire Notes Line
+	2050 2250 2850 2250
+Wire Notes Line
+	2850 2250 2850 1900
+Wire Notes Line
+	2850 1900 2050 1900
 $EndSCHEMATC
